Commit message: Improvement of some meshes.

File: ab2_description/urdf/ab2.urdf (robot description, URDF)
Before this commit: robot alphabot2, 6 links, 5 joints
Links:
- link base_link: geometry collision box size=0.14 0.14 0.05; visual mesh filename=package://ab2_description/meshes/glb/body.glb scale=1.0 1.0 1.0
- link wheel_left_link: geometry collision cylinder length=0.019 radius=0.021; visual mesh filename=package://ab2_description/meshes/glb/wheel.glb scale=1.0 1.0 1.0
- link wheel_right_link: geometry collision cylinder length=0.019 radius=0.021; visual mesh filename=package://ab2_description/meshes/glb/wheel.glb scale=1.0 1.0 1.0
Joints:
- joint base_joint: origin xyz=0.0 0.0 0.01 rpy=0 0 0 -> xyz=0 0 0 rpy=0 0 0
- joint wheel_right_joint: origin xyz=0.0425 0 0 rpy=0 3.14 0 -> xyz=0.0425 0 0 rpy=0 0 0

Commit message: Added Gazebo setup

File: ab2_description/urdf/ab2.urdf (robot description, URDF)
Before this commit: robot alphabot2, 6 links, 5 joints
Links:
- link base_link: geometry collision box size=0.14 0.14 0.05; visual mesh filename=package://ab2_description/meshes/dae/body.dae scale=1.0 1.0 1.0
- link wheel_left_link: geometry collision cylinder length=0.019 radius=0.021; visual mesh filename=package://ab2_description/meshes/dae/wheel.dae scale=1.0 1.0 1.0
- link wheel_right_link: geometry collision cylinder length=0.019 radius=0.021; visual mesh filename=package://ab2_description/meshes/dae/wheel.dae scale=1.0 1.0 1.0
Joints:
- joint base_joint: origin xyz=0 0 0 rpy=0 0 0 -> xyz=0 0 0 rpy=0 0 -1.5708

Commit message: Updated Alphabot2 models

File: ab2_description/urdf/ab2.urdf (robot description, URDF)
Before this commit: robot alphabot2, 6 links, 5 joints
Joints:
- joint wheel_left_joint: origin xyz=-0.0425 0 0 rpy=0 0 0 -> xyz=-0.044 0 0 rpy=0 0 0
- joint wheel_right_joint: origin xyz=0.0425 0 0 rpy=0 0 0 -> xyz=0.044 0 0 rpy=0 0 0

Commit message: Modified models

File: ab2_description/urdf/ab2.urdf (robot description, URDF)
Before this commit: robot alphabot2, 6 links, 5 joints
Links:
- added link landing_link
- link base_link: mass 0.50000000 -> 0.54000000; geometry collision box size=0.14 0.14 0.065; visual mesh filename=package://ab2_description/meshes/dae/body.dae scale=1.0 1.0 1.0
Joints:
- added joint landing_joint: type fixed, parent base_link, child landing_link, origin xyz=0 0 0.053 rpy=0 0 0
